File: pcb/pcb_left/pcb.kicad_sch (KiCad schematic)
At the start: 62 parts, among them J1 OLED_128x32, U1 Nice_Nano_V2

Commit message: Upadate v1.00
Parts:
- renumbered D1_L to D1_L1, S1_L to S1
Changed lines of the file:
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@@
 		(dnp no)
 		(fields_autoplaced yes)
-		(property "Reference" "D1_L"
+		(property "Reference" "D1_L1"
 			(at 160.02 55.8799 90)
 			(effects
@@
 			(project ""
 				(path "/9726f12a-2909-400c-a1f8-d834faf6b0fb"
-					(reference "D1_L")
+					(reference "D1_L1")
 					(unit 1)
 				)
@@
 		(dnp no)
 		(fields_autoplaced yes)
-		(property "Reference" "S1_L"
+		(property "Reference" "S1"
 			(at 154.94 43.18 0)
 			(effects
@@
 			(project ""
 				(path "/9726f12a-2909-400c-a1f8-d834faf6b0fb"
-					(reference "S1_L")
-					(unit 1)
-				)
+					(reference "S1")
+					(unit 1)
+				)
