File: pcb/PCB_Production/PCB_Production.kicad_pcb (KiCad board)
At the start: 2 copper layers, 339.5 x 112 mm, 123 parts, among them J1 OLED_128x32, U1 Nice_Nano_V2

Commit message: Upadate v1.00
Parts:
- removed the D1 at (-9.96, 51.8)
- removed the D1 at (290.1, 48.1)
- removed the D10 at (252.1, 61.6)
- removed the D10 at (28.0, 65.2)
- removed the D11 at (233.1, 61.4)
- removed the D11 at (47.0, 65.0)
- removed the D12 at (214.2, 69.0)
- removed the D12 at (65.9, 72.6)
- removed the D13 at (84.8, 72.5)
- removed the D13 at (195.3, 68.8)
- removed the D14 at (103.2, 72.3)
- removed the D14 at (176.9, 68.6)
- removed the D15 at (-9.91, 89.5)
- removed the D15 at (290.0, 85.9)
- removed the D16 at (271.2, 86.0)
- removed the D16 at (8.91, 89.7)
- removed the D17 at (252.0, 80.5)
- removed the D17 at (28.1, 84.2)
- removed the D18 at (47.0, 84.0)
- removed the D18 at (233.1, 80.3)
- removed the D19 at (65.9, 84.0)
- removed the D19 at (214.2, 80.4)
- removed the D2 at (9.04, 51.8)
- removed the D2 at (271.1, 48.2)
- removed the D20 at (195.2, 86.0)
- removed the D20 at (84.9, 89.6)
- removed the D21 at (103.0, 91.9)
- removed the D21 at (177.1, 88.2)
- removed the D22 at (-9.96, 108.7)
- removed the D22 at (290.1, 105.0)
- removed the D23 at (9.16, 108.5)
- removed the D23 at (270.9, 104.9)
- removed the D24 at (252.0, 99.5)
- removed the D24 at (28.1, 103.2)
- removed the D25 at (46.9, 103.0)
- removed the D25 at (233.2, 99.3)
- removed the D26 at (214.3, 99.5)
- removed the D26 at (65.8, 103.1)
- removed the D27 at (195.1, 105.0)
- removed the D27 at (85.0, 108.7)
- removed the D28 at (57.6, 133.1)
- removed the D28 at (222.5, 129.5)
- removed the D29 at (199.9, 129.5)
- removed the D29 at (80.2, 133.2)
- removed the D3 at (28.1, 46.2)
- removed the D3 at (252.0, 42.6)
- removed the D30 at (195.1, 110.6)
- removed the D30 at (85.0, 114.3)
- removed the D4 at (233.1, 42.5)
- removed the D4 at (47.0, 46.2)
- removed the D5 at (214.2, 48.6)
- removed the D5 at (65.9, 52.3)
- removed the D6 at (84.8, 57.9)
- removed the D6 at (195.3, 54.2)
- removed the D7 at (176.8, 54.2)
- removed the D7 at (103.3, 57.9)
- removed the D8 at (-9.91, 70.8)
- removed the D8 at (290.0, 67.1)
- removed the D9 at (9.02, 70.8)
- removed the D9 at (271.1, 67.2)
- removed the S1 at (299.6, 50.3)
- removed the S1 at (-19.5, 54.0)
- removed the S10 at (18.5, 67.4)
- removed the S10 at (261.6, 63.8)
- removed the S11 at (37.6, 65.3)
- removed the S11 at (242.5, 61.6)
- removed the S12 at (223.7, 63.9)
- removed the S12 at (56.4, 67.5)
- removed the S13 at (75.3, 73.0)
- removed the S13 at (204.8, 69.3)
- removed the S14 at (94.3, 75.3)
- removed the S14 at (185.8, 71.7)
- removed the S15 at (-19.5, 91.8)
- removed the S15 at (299.6, 88.2)
- removed the S16 at (-0.48, 91.8)
- removed the S16 at (280.6, 88.2)
- removed the S17 at (18.5, 86.3)
- removed the S17 at (261.6, 82.6)
- removed the S18 at (37.6, 84.2)
- removed the S18 at (242.5, 80.5)
- removed the S19 at (223.7, 82.8)
- removed the S19 at (56.4, 86.4)
- removed the S2 at (280.6, 50.4)
- removed the S2 at (-0.48, 54.0)
- removed the S20 at (204.8, 88.2)
- removed the S20 at (75.3, 91.8)
- removed the S21 at (94.3, 94.2)
- removed the S21 at (185.8, 90.5)
- removed the S22 at (-19.5, 110.8)
- removed the S22 at (299.6, 107.2)
- removed the S23 at (280.6, 107.2)
- removed the S23 at (-0.48, 110.8)
- removed the S24 at (261.6, 101.6)
- removed the S24 at (18.5, 105.3)
- removed the S25 at (242.5, 99.5)
- removed the S25 at (37.6, 103.2)
- removed the S26 at (223.7, 101.8)
- removed the S26 at (56.4, 105.4)
- removed the S27 at (204.8, 107.1)
- removed the S27 at (75.3, 110.8)
- removed the S28 at (232.9, 127.9)
- removed the S28 at (47.2, 131.6)
- removed the S29 at (69.2, 133.3)
- removed the S29 at (210.9, 129.6)
- removed the S3 at (261.5, 44.8)
- removed the S3 at (18.6, 48.5)
- removed the S30 at (92.6, 127.7)
- removed the S30 at (187.5, 124.1)
- removed the S4 at (37.6, 46.3)
- removed the S4 at (242.5, 42.6)
- removed the S5 at (223.7, 44.9)
- removed the S5 at (56.4, 48.5)
- removed the S6 at (204.8, 50.3)
- removed the S6 at (75.3, 54.0)
- removed the S7 at (185.8, 52.7)
- removed the S7 at (94.3, 56.4)
- removed the S8 at (-19.5, 73.0)
- removed the S8 at (299.6, 69.3)
- removed the S9 at (-0.48, 73.0)
- removed the S9 at (280.6, 69.3)
- removed the U1 at (163.9, 58.5)
- removed the U1 at (116.2, 62.0)
- added D1: Diode, Diode_SMD:D_SOD-123, B.Cu at (-77.8, 58.1)
- added D1: Diode, Diode_SMD:D_SOD-123, B.Cu at (201.4, 57.9)
- added D10: Diode, Diode_SMD:D_SOD-123, B.Cu at (163.4, 71.3)
- added D10: Diode, Diode_SMD:D_SOD-123, B.Cu at (-39.8, 71.5)
- added D11: Diode, Diode_SMD:D_SOD-123, B.Cu at (-20.8, 71.3)
- added D11: Diode, Diode_SMD:D_SOD-123, B.Cu at (144.4, 71.1)
- added D12: Diode, Diode_SMD:D_SOD-123, B.Cu at (125.5, 78.7)
- added D12: Diode, Diode_SMD:D_SOD-123, B.Cu at (-1.93, 78.9)
- added D13: Diode, Diode_SMD:D_SOD-123, B.Cu at (17.0, 78.7)
- added D13: Diode, Diode_SMD:D_SOD-123, B.Cu at (106.6, 78.6)
- added D14: Diode, Diode_SMD:D_SOD-123, B.Cu at (88.2, 78.4)
- added D14: Diode, Diode_SMD:D_SOD-123, B.Cu at (35.4, 78.5)
- added D15: Diode, Diode_SMD:D_SOD-123, B.Cu at (-77.8, 95.8)
- added D15: Diode, Diode_SMD:D_SOD-123, B.Cu at (201.4, 95.6)
- added D16: Diode, Diode_SMD:D_SOD-123, B.Cu at (-58.9, 96.0)
- added D16: Diode, Diode_SMD:D_SOD-123, B.Cu at (182.5, 95.8)
- added D17: Diode, Diode_SMD:D_SOD-123, B.Cu at (-39.8, 90.4)
- added D17: Diode, Diode_SMD:D_SOD-123, B.Cu at (163.4, 90.2)
- added D18: Diode, Diode_SMD:D_SOD-123, B.Cu at (144.4, 90.1)
- added D18: Diode, Diode_SMD:D_SOD-123, B.Cu at (-20.8, 90.3)
- added D19: Diode, Diode_SMD:D_SOD-123, B.Cu at (125.6, 90.1)
- added D19: Diode, Diode_SMD:D_SOD-123, B.Cu at (-1.95, 90.3)
- added D2: Diode, Diode_SMD:D_SOD-123, B.Cu at (-58.8, 58.1)
- added D2: Diode, Diode_SMD:D_SOD-123, B.Cu at (182.4, 57.9)
- added D20: Diode, Diode_SMD:D_SOD-123, B.Cu at (106.6, 95.7)
- added D20: Diode, Diode_SMD:D_SOD-123, B.Cu at (17.0, 95.9)
- added D21: Diode, Diode_SMD:D_SOD-123, B.Cu at (88.4, 98.0)
- added D21: Diode, Diode_SMD:D_SOD-123, B.Cu at (35.2, 98.1)
- added D22: Diode, Diode_SMD:D_SOD-123, B.Cu at (201.4, 114.7)
- added D22: Diode, Diode_SMD:D_SOD-123, B.Cu at (-77.8, 114.9)
- added D23: Diode, Diode_SMD:D_SOD-123, B.Cu at (-58.7, 114.8)
- added D23: Diode, Diode_SMD:D_SOD-123, B.Cu at (182.3, 114.6)
- added D24: Diode, Diode_SMD:D_SOD-123, B.Cu at (163.3, 109.3)
- added D24: Diode, Diode_SMD:D_SOD-123, B.Cu at (-39.7, 109.4)
- added D25: Diode, Diode_SMD:D_SOD-123, B.Cu at (-20.9, 109.2)
- added D25: Diode, Diode_SMD:D_SOD-123, B.Cu at (144.6, 109.1)
- added D26: Diode, Diode_SMD:D_SOD-123, B.Cu at (-2.05, 109.4)
- added D26: Diode, Diode_SMD:D_SOD-123, B.Cu at (125.7, 109.2)
- added D27: Diode, Diode_SMD:D_SOD-123, B.Cu at (17.2, 114.9)
- added D27: Diode, Diode_SMD:D_SOD-123, B.Cu at (106.4, 114.7)
- added D28: Diode, Diode_SMD:D_SOD-123, B.Cu at (-10.3, 139.4)
- added D28: Diode, Diode_SMD:D_SOD-123, B.Cu at (133.9, 139.2)
- added D29: Diode, Diode_SMD:D_SOD-123, B.Cu at (12.3, 139.4)
- added D29: Diode, Diode_SMD:D_SOD-123, B.Cu at (111.3, 139.2)
- added D3: Diode, Diode_SMD:D_SOD-123, B.Cu at (-39.7, 52.5)
- added D3: Diode, Diode_SMD:D_SOD-123, B.Cu at (163.3, 52.3)
- added D30: Diode, Diode_SMD:D_SOD-123, B.Cu at (17.2, 120.5)
- added D30: Diode, Diode_SMD:D_SOD-123, B.Cu at (106.4, 120.4)
- added D4: Diode, Diode_SMD:D_SOD-123, B.Cu at (-20.9, 52.4)
- added D4: Diode, Diode_SMD:D_SOD-123, B.Cu at (144.5, 52.3)
- added D5: Diode, Diode_SMD:D_SOD-123, B.Cu at (125.6, 58.4)
- added D5: Diode, Diode_SMD:D_SOD-123, B.Cu at (-1.95, 58.6)
- added D6: Diode, Diode_SMD:D_SOD-123, B.Cu at (106.6, 63.9)
- added D6: Diode, Diode_SMD:D_SOD-123, B.Cu at (17.0, 64.1)
- added D7: Diode, Diode_SMD:D_SOD-123, B.Cu at (35.5, 64.1)
- added D7: Diode, Diode_SMD:D_SOD-123, B.Cu at (88.2, 64.0)
- added D8: Diode, Diode_SMD:D_SOD-123, B.Cu at (201.4, 76.8)
- added D8: Diode, Diode_SMD:D_SOD-123, B.Cu at (-77.8, 77.0)
- added D9: Diode, Diode_SMD:D_SOD-123, B.Cu at (182.4, 76.9)
- added D9: Diode, Diode_SMD:D_SOD-123, B.Cu at (-58.8, 77.1)
- added S1: Keyswitch, ScottoKeebs_Choc:Choc_V2, F.Cu at (-87.3, 60.2)
- added S1: Keyswitch, ScottoKeebs_Choc:Choc_V2, F.Cu at (210.9, 60.0)
- added S10: Keyswitch, ScottoKeebs_Choc:Choc_V2, F.Cu at (172.9, 73.5)
- added S10: Keyswitch, ScottoKeebs_Choc:Choc_V2, F.Cu at (-49.3, 73.7)
- added S11: Keyswitch, ScottoKeebs_Choc:Choc_V2, F.Cu at (153.8, 71.4)
- added S11: Keyswitch, ScottoKeebs_Choc:Choc_V2, F.Cu at (-30.2, 71.6)
- added S12: Keyswitch, ScottoKeebs_Choc:Choc_V2, F.Cu at (135.1, 73.6)
- added S12: Keyswitch, ScottoKeebs_Choc:Choc_V2, F.Cu at (-11.5, 73.8)
- added S13: Keyswitch, ScottoKeebs_Choc:Choc_V2, F.Cu at (116.1, 79.0)
- added S13: Keyswitch, ScottoKeebs_Choc:Choc_V2, F.Cu at (7.47, 79.2)
- added S14: Keyswitch, ScottoKeebs_Choc:Choc_V2, F.Cu at (97.2, 81.4)
- added S14: Keyswitch, ScottoKeebs_Choc:Choc_V2, F.Cu at (26.4, 81.6)
- added S15: Keyswitch, ScottoKeebs_Choc:Choc_V2, F.Cu at (210.9, 97.9)
- added S15: Keyswitch, ScottoKeebs_Choc:Choc_V2, F.Cu at (-87.3, 98.1)
- added S16: Keyswitch, ScottoKeebs_Choc:Choc_V2, F.Cu at (-68.3, 98.1)
- added S16: Keyswitch, ScottoKeebs_Choc:Choc_V2, F.Cu at (191.9, 97.9)
- added S17: Keyswitch, ScottoKeebs_Choc:Choc_V2, F.Cu at (-49.3, 92.5)
- added S17: Keyswitch, ScottoKeebs_Choc:Choc_V2, F.Cu at (172.9, 92.4)
- added S18: Keyswitch, ScottoKeebs_Choc:Choc_V2, F.Cu at (153.8, 90.2)
- added S18: Keyswitch, ScottoKeebs_Choc:Choc_V2, F.Cu at (-30.2, 90.4)
- added S19: Keyswitch, ScottoKeebs_Choc:Choc_V2, F.Cu at (135.1, 92.5)
- added S19: Keyswitch, ScottoKeebs_Choc:Choc_V2, F.Cu at (-11.5, 92.7)
- added S2: Keyswitch, ScottoKeebs_Choc:Choc_V2, F.Cu at (191.9, 60.1)
- added S2: Keyswitch, ScottoKeebs_Choc:Choc_V2, F.Cu at (-68.3, 60.3)
- added S20: Keyswitch, ScottoKeebs_Choc:Choc_V2, F.Cu at (116.1, 97.9)
- added S20: Keyswitch, ScottoKeebs_Choc:Choc_V2, F.Cu at (7.47, 98.1)
- added S21: Keyswitch, ScottoKeebs_Choc:Choc_V2, F.Cu at (97.1, 100.2)
- added S21: Keyswitch, ScottoKeebs_Choc:Choc_V2, F.Cu at (26.5, 100.4)
- added S22: Keyswitch, ScottoKeebs_Choc:Choc_V2, F.Cu at (-87.3, 117.1)
- added S22: Keyswitch, ScottoKeebs_Choc:Choc_V2, F.Cu at (210.9, 116.9)
- added S23: Keyswitch, ScottoKeebs_Choc:Choc_V2, F.Cu at (-68.3, 117.1)
- added S23: Keyswitch, ScottoKeebs_Choc:Choc_V2, F.Cu at (191.9, 116.9)
- added S24: Keyswitch, ScottoKeebs_Choc:Choc_V2, F.Cu at (172.9, 111.4)
- added S24: Keyswitch, ScottoKeebs_Choc:Choc_V2, F.Cu at (-49.3, 111.5)
- added S25: Keyswitch, ScottoKeebs_Choc:Choc_V2, F.Cu at (-30.2, 109.4)
- added S25: Keyswitch, ScottoKeebs_Choc:Choc_V2, F.Cu at (153.8, 109.2)
- added S26: Keyswitch, ScottoKeebs_Choc:Choc_V2, F.Cu at (-11.5, 111.7)
- added S26: Keyswitch, ScottoKeebs_Choc:Choc_V2, F.Cu at (135.1, 111.5)
- added S27: Keyswitch, ScottoKeebs_Choc:Choc_V2, F.Cu at (116.1, 116.9)
- added S27: Keyswitch, ScottoKeebs_Choc:Choc_V2, F.Cu at (7.47, 117.0)
- added S28: Keyswitch, ScottoKeebs_Choc:Choc_V2, F.Cu at (-20.6, 137.8)
- added S28: Keyswitch, ScottoKeebs_Choc:Choc_V2, F.Cu at (144.2, 137.6)
- added S29: Keyswitch, ScottoKeebs_Choc:Choc_V2, F.Cu at (122.2, 139.4)
- added S29: Keyswitch, ScottoKeebs_Choc:Choc_V2, F.Cu at (1.41, 139.6)
- added S3: Keyswitch, ScottoKeebs_Choc:Choc_V2, F.Cu at (172.9, 54.5)
- added S30: Keyswitch, ScottoKeebs_Choc:Choc_V2, F.Cu at (98.8, 133.8)
- added S30: Keyswitch, ScottoKeebs_Choc:Choc_V2, F.Cu at (24.8, 134.0)
- added S4: Keyswitch, ScottoKeebs_Choc:Choc_V2, F.Cu at (-49.3, 54.7)
- added S4: Keyswitch, ScottoKeebs_Choc:Choc_V2, F.Cu at (153.8, 52.4)
- added S4: Keyswitch, ScottoKeebs_Choc:Choc_V2, F.Cu at (-30.2, 52.6)
- added S5: Keyswitch, ScottoKeebs_Choc:Choc_V2, F.Cu at (135.1, 54.6)
- added S5: Keyswitch, ScottoKeebs_Choc:Choc_V2, F.Cu at (-11.5, 54.8)
- added S6: Keyswitch, ScottoKeebs_Choc:Choc_V2, F.Cu at (116.1, 60.0)
- added S6: Keyswitch, ScottoKeebs_Choc:Choc_V2, F.Cu at (7.47, 60.2)
- added S7: Keyswitch, ScottoKeebs_Choc:Choc_V2, F.Cu at (97.1, 62.4)
- added S7: Keyswitch, ScottoKeebs_Choc:Choc_V2, F.Cu at (26.5, 62.6)
- added S8: Keyswitch, ScottoKeebs_Choc:Choc_V2, F.Cu at (-87.3, 79.2)
- added S8: Keyswitch, ScottoKeebs_Choc:Choc_V2, F.Cu at (210.9, 79.0)
- added S9: Keyswitch, ScottoKeebs_Choc:Choc_V2, F.Cu at (-68.3, 79.3)
- added S9: Keyswitch, ScottoKeebs_Choc:Choc_V2, F.Cu at (191.9, 79.1)
- added U1: Nice_Nano_V2, ScottoKeebs_MCU:Nice_Nano_V2, B.Cu at (75.3, 68.3)
- added U1: Nice_Nano_V2, ScottoKeebs_MCU:Nice_Nano_V2, B.Cu at (48.4, 68.3)
- moved J1 68.1 mm to (54.5, 84.9)
Routing:
- net Col_0: track 110.4 -> 112.8 mm
- net Col_1: track 144.0 -> 146.4 mm
- net Net-(D29-A): track 23.5 -> 21.9 mm
- net Net-(D30-A): track 32.6 -> 31.1 mm
Other:
- board size 339.5 x 112 mm -> 316.3 x 108.6 mm

Commit message: Upadate v1.00
Parts:
- removed the D1 at (-77.8, 58.1)
- removed the D1 at (201.4, 57.9)
- removed the D10 at (163.4, 71.3)
- removed the D10 at (-39.8, 71.5)
- removed the D11 at (-20.8, 71.3)
- removed the D11 at (144.4, 71.1)
- removed the D12 at (125.5, 78.7)
- removed the D12 at (-1.93, 78.9)
- removed the D13 at (17.0, 78.7)
- removed the D13 at (106.6, 78.6)
- removed the D14 at (88.2, 78.4)
- removed the D14 at (35.4, 78.5)
- removed the D15 at (-77.8, 95.8)
- removed the D15 at (201.4, 95.6)
- removed the D16 at (-58.9, 96.0)
- removed the D16 at (182.5, 95.8)
- removed the D17 at (-39.8, 90.4)
- removed the D17 at (163.4, 90.2)
- removed the D18 at (144.4, 90.1)
- removed the D18 at (-20.8, 90.3)
- removed the D19 at (125.6, 90.1)
- removed the D19 at (-1.95, 90.3)
- removed the D2 at (-58.8, 58.1)
- removed the D2 at (182.4, 57.9)
- removed the D20 at (106.6, 95.7)
- removed the D20 at (17.0, 95.9)
- removed the D21 at (88.4, 98.0)
- removed the D21 at (35.2, 98.1)
- removed the D22 at (201.4, 114.7)
- removed the D22 at (-77.8, 114.9)
- removed the D23 at (-58.7, 114.8)
- removed the D23 at (182.3, 114.6)
- removed the D24 at (163.3, 109.3)
- removed the D24 at (-39.7, 109.4)
- removed the D25 at (-20.9, 109.2)
- removed the D25 at (144.6, 109.1)
- removed the D26 at (-2.05, 109.4)
- removed the D26 at (125.7, 109.2)
- removed the D27 at (17.2, 114.9)
- removed the D27 at (106.4, 114.7)
- removed the D28 at (-10.3, 139.4)
- removed the D28 at (133.9, 139.2)
- removed the D29 at (12.3, 139.4)
- removed the D29 at (111.3, 139.2)
- removed the D3 at (-39.7, 52.5)
- removed the D3 at (163.3, 52.3)
- removed the D30 at (17.2, 120.5)
- removed the D30 at (106.4, 120.4)
- removed the D4 at (-20.9, 52.4)
- removed the D4 at (144.5, 52.3)
- removed the D5 at (125.6, 58.4)
- removed the D5 at (-1.95, 58.6)
- removed the D6 at (106.6, 63.9)
- removed the D6 at (17.0, 64.1)
- removed the D7 at (35.5, 64.1)
- removed the D7 at (88.2, 64.0)
- removed the D8 at (201.4, 76.8)
- removed the D8 at (-77.8, 77.0)
- removed the D9 at (182.4, 76.9)
- removed the D9 at (-58.8, 77.1)
- removed the S1 at (-87.3, 60.2)
- removed the S1 at (210.9, 60.0)
- removed the S10 at (172.9, 73.5)
- removed the S10 at (-49.3, 73.7)
- removed the S11 at (153.8, 71.4)
- removed the S11 at (-30.2, 71.6)
- removed the S12 at (135.1, 73.6)
- removed the S12 at (-11.5, 73.8)
- removed the S13 at (116.1, 79.0)
- removed the S13 at (7.47, 79.2)
- removed the S14 at (97.2, 81.4)
- removed the S14 at (26.4, 81.6)
- removed the S15 at (210.9, 97.9)
- removed the S15 at (-87.3, 98.1)
- removed the S16 at (-68.3, 98.1)
- removed the S16 at (191.9, 97.9)
- removed the S17 at (-49.3, 92.5)
- removed the S17 at (172.9, 92.4)
- removed the S18 at (153.8, 90.2)
- removed the S18 at (-30.2, 90.4)
- removed the S19 at (135.1, 92.5)
- removed the S19 at (-11.5, 92.7)
- removed the S2 at (191.9, 60.1)
- removed the S2 at (-68.3, 60.3)
- removed the S20 at (116.1, 97.9)
- removed the S20 at (7.47, 98.1)
- removed the S21 at (97.1, 100.2)
- removed the S21 at (26.5, 100.4)
- removed the S22 at (-87.3, 117.1)
- removed the S22 at (210.9, 116.9)
- removed the S23 at (-68.3, 117.1)
- removed the S23 at (191.9, 116.9)
- removed the S24 at (172.9, 111.4)
- removed the S24 at (-49.3, 111.5)
- removed the S25 at (-30.2, 109.4)
- removed the S25 at (153.8, 109.2)
- removed the S26 at (-11.5, 111.7)
- removed the S26 at (135.1, 111.5)
- removed the S27 at (116.1, 116.9)
- removed the S27 at (7.47, 117.0)
- removed the S28 at (-20.6, 137.8)
- removed the S28 at (144.2, 137.6)
- removed the S29 at (122.2, 139.4)
- removed the S29 at (1.41, 139.6)
- removed the S30 at (98.8, 133.8)
- removed the S30 at (24.8, 134.0)
- removed the S4 at (-49.3, 54.7)
- removed the S4 at (153.8, 52.4)
- removed the S4 at (-30.2, 52.6)
- removed the S5 at (135.1, 54.6)
- removed the S5 at (-11.5, 54.8)
- removed the S6 at (116.1, 60.0)
- removed the S6 at (7.47, 60.2)
- removed the S7 at (97.1, 62.4)
- removed the S7 at (26.5, 62.6)
- removed the S8 at (-87.3, 79.2)
- removed the S8 at (210.9, 79.0)
- removed the S9 at (-68.3, 79.3)
- removed the S9 at (191.9, 79.1)
- removed the U1 at (75.3, 68.3)
- removed the U1 at (48.4, 68.3)
- added D1: Diode, Diode_SMD:D_SOD-123, B.Cu at (252.3, 58.0)
- added D1: Diode, Diode_SMD:D_SOD-123, B.Cu at (-22.0, 58.0)
- added D10: Diode, Diode_SMD:D_SOD-123, B.Cu at (214.3, 71.5)
- added D10: Diode, Diode_SMD:D_SOD-123, B.Cu at (16.0, 71.4)
- added D11: Diode, Diode_SMD:D_SOD-123, B.Cu at (195.3, 71.2)
- added D11: Diode, Diode_SMD:D_SOD-123, B.Cu at (35.0, 71.2)
- added D12: Diode, Diode_SMD:D_SOD-123, B.Cu at (53.9, 78.8)
- added D12: Diode, Diode_SMD:D_SOD-123, B.Cu at (176.5, 78.8)
- added D13: Diode, Diode_SMD:D_SOD-123, B.Cu at (157.6, 78.7)
- added D13: Diode, Diode_SMD:D_SOD-123, B.Cu at (72.8, 78.7)
- added D14: Diode, Diode_SMD:D_SOD-123, B.Cu at (139.2, 78.5)
- added D14: Diode, Diode_SMD:D_SOD-123, B.Cu at (91.2, 78.5)
- added D15: Diode, Diode_SMD:D_SOD-123, B.Cu at (252.3, 95.8)
- added D15: Diode, Diode_SMD:D_SOD-123, B.Cu at (-21.9, 95.7)
- added D16: Diode, Diode_SMD:D_SOD-123, B.Cu at (-3.10, 95.9)
- added D16: Diode, Diode_SMD:D_SOD-123, B.Cu at (233.5, 95.9)
- added D17: Diode, Diode_SMD:D_SOD-123, B.Cu at (214.3, 90.4)
- added D17: Diode, Diode_SMD:D_SOD-123, B.Cu at (16.1, 90.3)
- added D18: Diode, Diode_SMD:D_SOD-123, B.Cu at (35.0, 90.2)
- added D18: Diode, Diode_SMD:D_SOD-123, B.Cu at (195.4, 90.2)
- added D19: Diode, Diode_SMD:D_SOD-123, B.Cu at (53.9, 90.2)
- added D19: Diode, Diode_SMD:D_SOD-123, B.Cu at (176.5, 90.3)
- added D2: Diode, Diode_SMD:D_SOD-123, B.Cu at (-2.98, 58.0)
- added D2: Diode, Diode_SMD:D_SOD-123, B.Cu at (233.3, 58.0)
- added D20: Diode, Diode_SMD:D_SOD-123, B.Cu at (72.8, 95.8)
- added D20: Diode, Diode_SMD:D_SOD-123, B.Cu at (157.5, 95.8)
- added D21: Diode, Diode_SMD:D_SOD-123, B.Cu at (139.4, 98.1)
- added D21: Diode, Diode_SMD:D_SOD-123, B.Cu at (91.0, 98.1)
- added D22: Diode, Diode_SMD:D_SOD-123, B.Cu at (-22.0, 114.8)
- added D22: Diode, Diode_SMD:D_SOD-123, B.Cu at (252.3, 114.9)
- added D23: Diode, Diode_SMD:D_SOD-123, B.Cu at (233.2, 114.7)
- added D23: Diode, Diode_SMD:D_SOD-123, B.Cu at (-2.85, 114.7)
- added D24: Diode, Diode_SMD:D_SOD-123, B.Cu at (16.1, 109.4)
- added D24: Diode, Diode_SMD:D_SOD-123, B.Cu at (214.2, 109.4)
- added D25: Diode, Diode_SMD:D_SOD-123, B.Cu at (34.9, 109.2)
- added D25: Diode, Diode_SMD:D_SOD-123, B.Cu at (195.5, 109.2)
- added D26: Diode, Diode_SMD:D_SOD-123, B.Cu at (176.6, 109.3)
- added D26: Diode, Diode_SMD:D_SOD-123, B.Cu at (53.8, 109.3)
- added D27: Diode, Diode_SMD:D_SOD-123, B.Cu at (73.0, 114.8)
- added D27: Diode, Diode_SMD:D_SOD-123, B.Cu at (157.4, 114.9)
- added D28: Diode, Diode_SMD:D_SOD-123, B.Cu at (45.5, 139.3)
- added D28: Diode, Diode_SMD:D_SOD-123, B.Cu at (184.8, 139.3)
- added D29: Diode, Diode_SMD:D_SOD-123, B.Cu at (68.2, 139.3)
- added D29: Diode, Diode_SMD:D_SOD-123, B.Cu at (162.2, 139.4)
- added D3: Diode, Diode_SMD:D_SOD-123, B.Cu at (16.1, 52.4)
- added D3: Diode, Diode_SMD:D_SOD-123, B.Cu at (214.3, 52.5)
- added D30: Diode, Diode_SMD:D_SOD-123, B.Cu at (73.0, 120.5)
- added D30: Diode, Diode_SMD:D_SOD-123, B.Cu at (157.3, 120.5)
- added D4: Diode, Diode_SMD:D_SOD-123, B.Cu at (195.4, 52.4)
- added D4: Diode, Diode_SMD:D_SOD-123, B.Cu at (34.9, 52.4)
- added D5: Diode, Diode_SMD:D_SOD-123, B.Cu at (176.5, 58.5)
- added D5: Diode, Diode_SMD:D_SOD-123, B.Cu at (53.9, 58.5)
- added D6: Diode, Diode_SMD:D_SOD-123, B.Cu at (157.5, 64.1)
- added D6: Diode, Diode_SMD:D_SOD-123, B.Cu at (72.8, 64.0)
- added D7: Diode, Diode_SMD:D_SOD-123, B.Cu at (91.3, 64.1)
- added D7: Diode, Diode_SMD:D_SOD-123, B.Cu at (139.1, 64.1)
- added D8: Diode, Diode_SMD:D_SOD-123, B.Cu at (252.3, 77.0)
- added D8: Diode, Diode_SMD:D_SOD-123, B.Cu at (-21.9, 76.9)
- added D9: Diode, Diode_SMD:D_SOD-123, B.Cu at (233.4, 77.0)
- added D9: Diode, Diode_SMD:D_SOD-123, B.Cu at (-3.00, 77.0)
- added S1: Keyswitch, ScottoKeebs_Choc:Choc_V2, F.Cu at (-31.5, 60.1)
- added S1: Keyswitch, ScottoKeebs_Choc:Choc_V2, F.Cu at (261.9, 60.2)
- added S10: Keyswitch, ScottoKeebs_Choc:Choc_V2, F.Cu at (223.8, 73.6)
- added S10: Keyswitch, ScottoKeebs_Choc:Choc_V2, F.Cu at (6.52, 73.6)
- added S11: Keyswitch, ScottoKeebs_Choc:Choc_V2, F.Cu at (204.8, 71.5)
- added S11: Keyswitch, ScottoKeebs_Choc:Choc_V2, F.Cu at (25.6, 71.5)
- added S12: Keyswitch, ScottoKeebs_Choc:Choc_V2, F.Cu at (44.3, 73.7)
- added S12: Keyswitch, ScottoKeebs_Choc:Choc_V2, F.Cu at (186.0, 73.8)
- added S13: Keyswitch, ScottoKeebs_Choc:Choc_V2, F.Cu at (167.1, 79.2)
- added S13: Keyswitch, ScottoKeebs_Choc:Choc_V2, F.Cu at (63.3, 79.1)
- added S14: Keyswitch, ScottoKeebs_Choc:Choc_V2, F.Cu at (82.2, 81.5)
- added S14: Keyswitch, ScottoKeebs_Choc:Choc_V2, F.Cu at (148.1, 81.6)
- added S15: Keyswitch, ScottoKeebs_Choc:Choc_V2, F.Cu at (261.9, 98.0)
- added S15: Keyswitch, ScottoKeebs_Choc:Choc_V2, F.Cu at (-31.5, 98.0)
- added S16: Keyswitch, ScottoKeebs_Choc:Choc_V2, F.Cu at (242.9, 98.1)
- added S16: Keyswitch, ScottoKeebs_Choc:Choc_V2, F.Cu at (-12.5, 98.0)
- added S17: Keyswitch, ScottoKeebs_Choc:Choc_V2, F.Cu at (6.52, 92.5)
- added S17: Keyswitch, ScottoKeebs_Choc:Choc_V2, F.Cu at (223.8, 92.5)
- added S18: Keyswitch, ScottoKeebs_Choc:Choc_V2, F.Cu at (25.6, 90.3)
- added S18: Keyswitch, ScottoKeebs_Choc:Choc_V2, F.Cu at (204.8, 90.4)
- added S19: Keyswitch, ScottoKeebs_Choc:Choc_V2, F.Cu at (186.0, 92.6)
- added S19: Keyswitch, ScottoKeebs_Choc:Choc_V2, F.Cu at (44.3, 92.6)
- added S2: Keyswitch, ScottoKeebs_Choc:Choc_V2, F.Cu at (-12.5, 60.2)
- added S2: Keyswitch, ScottoKeebs_Choc:Choc_V2, F.Cu at (242.9, 60.2)
- added S20: Keyswitch, ScottoKeebs_Choc:Choc_V2, F.Cu at (167.1, 98.0)
- added S20: Keyswitch, ScottoKeebs_Choc:Choc_V2, F.Cu at (63.3, 98.0)
- added S21: Keyswitch, ScottoKeebs_Choc:Choc_V2, F.Cu at (82.3, 100.3)
- added S21: Keyswitch, ScottoKeebs_Choc:Choc_V2, F.Cu at (148.1, 100.4)
- added S22: Keyswitch, ScottoKeebs_Choc:Choc_V2, F.Cu at (261.9, 117.0)
- added S22: Keyswitch, ScottoKeebs_Choc:Choc_V2, F.Cu at (-31.5, 117.0)
- added S23: Keyswitch, ScottoKeebs_Choc:Choc_V2, F.Cu at (242.9, 117.1)
- added S23: Keyswitch, ScottoKeebs_Choc:Choc_V2, F.Cu at (-12.5, 117.0)
- added S24: Keyswitch, ScottoKeebs_Choc:Choc_V2, F.Cu at (6.52, 111.5)
- added S24: Keyswitch, ScottoKeebs_Choc:Choc_V2, F.Cu at (223.8, 111.5)
- added S25: Keyswitch, ScottoKeebs_Choc:Choc_V2, F.Cu at (204.8, 109.4)
- added S25: Keyswitch, ScottoKeebs_Choc:Choc_V2, F.Cu at (25.6, 109.3)
- added S26: Keyswitch, ScottoKeebs_Choc:Choc_V2, F.Cu at (44.3, 111.6)
- added S26: Keyswitch, ScottoKeebs_Choc:Choc_V2, F.Cu at (186.0, 111.6)
- added S27: Keyswitch, ScottoKeebs_Choc:Choc_V2, F.Cu at (63.3, 117.0)
- added S27: Keyswitch, ScottoKeebs_Choc:Choc_V2, F.Cu at (167.1, 117.0)
- added S28: Keyswitch, ScottoKeebs_Choc:Choc_V2, F.Cu at (195.2, 137.8)
- added S28: Keyswitch, ScottoKeebs_Choc:Choc_V2, F.Cu at (35.2, 137.7)
- added S29: Keyswitch, ScottoKeebs_Choc:Choc_V2, F.Cu at (173.1, 139.5)
- added S29: Keyswitch, ScottoKeebs_Choc:Choc_V2, F.Cu at (57.2, 139.5)
- added S30: Keyswitch, ScottoKeebs_Choc:Choc_V2, F.Cu at (80.6, 133.9)
- added S30: Keyswitch, ScottoKeebs_Choc:Choc_V2, F.Cu at (149.7, 134.0)
- added S4: Keyswitch, ScottoKeebs_Choc:Choc_V2, F.Cu at (204.8, 52.5)
- added S4: Keyswitch, ScottoKeebs_Choc:Choc_V2, F.Cu at (6.55, 54.6)
- added S4: Keyswitch, ScottoKeebs_Choc:Choc_V2, F.Cu at (25.6, 52.5)
- added S5: Keyswitch, ScottoKeebs_Choc:Choc_V2, F.Cu at (44.3, 54.7)
- added S5: Keyswitch, ScottoKeebs_Choc:Choc_V2, F.Cu at (186.0, 54.8)
- added S6: Keyswitch, ScottoKeebs_Choc:Choc_V2, F.Cu at (63.3, 60.1)
- added S6: Keyswitch, ScottoKeebs_Choc:Choc_V2, F.Cu at (167.1, 60.2)
- added S7: Keyswitch, ScottoKeebs_Choc:Choc_V2, F.Cu at (82.3, 62.5)
- added S7: Keyswitch, ScottoKeebs_Choc:Choc_V2, F.Cu at (148.1, 62.6)
- added S8: Keyswitch, ScottoKeebs_Choc:Choc_V2, F.Cu at (-31.5, 79.1)
- added S8: Keyswitch, ScottoKeebs_Choc:Choc_V2, F.Cu at (261.9, 79.2)
- added S9: Keyswitch, ScottoKeebs_Choc:Choc_V2, F.Cu at (242.9, 79.2)
- added S9: Keyswitch, ScottoKeebs_Choc:Choc_V2, F.Cu at (-12.5, 79.2)
- added U1: Nice_Nano_V2, ScottoKeebs_MCU:Nice_Nano_V2, B.Cu at (126.2, 68.4)
- added U1: Nice_Nano_V2, ScottoKeebs_MCU:Nice_Nano_V2, B.Cu at (104.2, 68.2)
- moved J1 55.8 mm to (110.3, 84.8)
- moved S3 50.9 mm to (223.8, 54.7)
Routing:
- net Row_3: track 267.5 -> 195.4 mm, vias 0 -> 2
- net Col_0: track 112.8 -> 110.6 mm, vias 0 -> 2
Other:
- board size 316.3 x 108.6 mm -> 311.2 x 108.4 mm
